File: CMP3_Amp.sch (EAGLE design)
At the start: 22 parts, among them J1 CONN_42.54_SCREW, J2 CONN_33.5_SCREW, Q2 DMG3404, U1 LTC2054, U2 LTC2054

Commit message: Initial layout of CMP3 Amp
Layout of CMP3 amp complete, requires review and gerber generation before being sent to fab
Parts:
- added TP1, TP2, TP3, TP4: TESTPOINTRCU, bschulz:TESTPOINTRCU
- renumbered U$3 to U4, U$6 to U5, U$8 to U3
Connections:
- net GND: now also TP4.P$1
- net SCL: now also U4.A2; no longer U4.A1
- net SCL_HV: now also U4.B2; no longer U4.B1
- net SDA: now also U4.A1; no longer U4.A2
- net SDA_HV: now also U4.B1; no longer U4.B2
- net VOUT_FILT: now also TP3.P$1
- net VOUT_GAIN: now also TP2.P$1
- net V_PYRO: now also TP1.P$1
